Commit message: Refactor code structure for improved readability and maintainability

File: delta_robot_description/models/NEWWW.sdf.xacro (robot description, xacro)
@@ -674,12 +674,8 @@
         <xacro:end_effector_pinion          n="1" relative_to="sts_circular_horn_1"/>
         <xacro:end_effector_pinion          n="2" relative_to="sts_circular_horn_2"/>
-        <link name="virtual_middle_shaft">
-            <self_collide>false</self_collide>
-            <pose relative_to="end_effector_pinion_1">0 0.028 0 ${-pi/2} 0 ${-pi/2}</pose>
-        </link>
         <!-- Middle shaft — driven (differential_T_joint child) -->
         <link name="middle_shaft">
             <self_collide>false</self_collide>
-            <pose relative_to="virtual_middle_shaft">0 0.0070 0 0 0 0</pose>
+            <pose relative_to="end_effector_pinion_1">0 0.028 -0.0070 ${-pi/2} 0 ${-pi/2}</pose>
             <inertial>
                 <mass>0.0162455078</mass>
@@ -816,11 +812,10 @@
         <xacro:fixed_joint    name="base_plate_to_side_plate_1"   parent="end_effector_base_plate" child="end_effector_side_plate_1"/>
         <xacro:fixed_joint    name="base_plate_to_side_plate_2"   parent="end_effector_base_plate" child="end_effector_side_plate_2"/>
-        <xacro:revolute_joint name="differential_T_joint"         parent="end_effector_base_plate" child="virtual_middle_shaft"           ax="-1" ay="0"  az="0"/>
+        <xacro:revolute_joint name="differential_T_joint"         parent="end_effector_base_plate" child="middle_shaft"           ax="1" ay="0"  az="0"/>
         <xacro:fixed_joint    name="side_plate_1_to_diff_servo_1" parent="end_effector_side_plate_1" child="differential_servo_1"/>
         <xacro:fixed_joint    name="side_plate_2_to_diff_servo_2" parent="end_effector_side_plate_2" child="differential_servo_2"/>
-        <xacro:fixed_joint    name="virtual_middle_shaft_to_middle_shaft"     parent="virtual_middle_shaft"     child="middle_shaft"/>
-        <xacro:revolute_joint name="differential_EE_joint"        parent="middle_shaft"            child="bevel_gear_ee"          ax="0" ay="1" az="0"/>
-        <xacro:revolute_joint name="differential_pinion_joint_1"  parent="differential_servo_1"    child="sts_circular_horn_1"    ax="1" ay="0"  az="0"/>
-        <xacro:revolute_joint name="differential_pinion_joint_2"  parent="differential_servo_2"    child="sts_circular_horn_2"    ax="1" ay="0"  az="0"/>
+        <xacro:revolute_joint name="differential_EE_joint"        parent="middle_shaft"            child="bevel_gear_ee"          ax="0" ay="-1" az="0"/>
+        <xacro:revolute_joint name="differential_pinion_joint_1"  parent="differential_servo_1"    child="sts_circular_horn_1"    ax="-1" ay="0"  az="0"/>
+        <xacro:revolute_joint name="differential_pinion_joint_2"  parent="differential_servo_2"    child="sts_circular_horn_2"    ax="-1" ay="0"  az="0"/>
         <xacro:fixed_joint    name="sts_horn_1_to_ee_pinion_1"    parent="sts_circular_horn_1"     child="end_effector_pinion_1"/>
         <xacro:fixed_joint    name="sts_horn_2_to_ee_pinion_2"    parent="sts_circular_horn_2"     child="end_effector_pinion_2"/>

File: delta_robot_description/models/model_high.sdf copy.xacro (robot description, xacro)
@@ -1,11 +1,8 @@
 <?xml version='1.0' encoding='utf-8'?>
 <sdf xmlns:xacro="http://www.ros.org/wiki/xacro" version="1.7">
-    <!-- ══════════════════════════════════════════════════════════
-         PROPERTIES
-    ══════════════════════════════════════════════════════════ -->
+    <!-- PROPERTIES-->
+    <!-- Mesh package base-path. -->
     <xacro:property name="meshes" value="package://delta_robot_description/meshes"/>
-    <!-- ══════════════════════════════════════════════════════════
-         MATERIAL MACROS
-    ══════════════════════════════════════════════════════════ -->
+    <!-- MATERIAL MACROS -->
     <xacro:macro name="material_aluminium">
         <material>
@@ -64,9 +61,5 @@
         </material>
     </xacro:macro>
-    <!-- ══════════════════════════════════════════════════════════
-         INERTIA MACROS
-         Cross-terms (ixy/ixz/iyz) with |value| < 1e-9 are zeroed.
-         Negligible CoM pose offsets below the same threshold are also zeroed.
-    ══════════════════════════════════════════════════════════ -->
+    <!-- INERTIA MACROS -->
     <!-- Servo mount (×3) -->
     <xacro:macro name="inertial_servo_mount">
@@ -99,5 +92,5 @@
         </inertial>
     </xacro:macro>
-    <!-- Servo horn / free-horn (×6) — driven (motor_joint_1/2/3 children) -->
+    <!-- Servo horn / free-horn (×6) -->
     <xacro:macro name="inertial_servo_horn">
         <inertial>
@@ -129,5 +122,5 @@
         </inertial>
     </xacro:macro>
-    <!-- Upper pivot arm (×3) -->
+    <!-- Upper pivot arm — pivot_arm_1 / 2 / 3 -->
     <xacro:macro name="inertial_pivot_arm_upper">
         <inertial>
@@ -144,5 +137,5 @@
         </inertial>
     </xacro:macro>
-    <!-- Upper rod-cap (×6) -->
+    <!-- Upper rod-cap — rod_cap_1 … rod_cap_6 -->
     <xacro:macro name="inertial_rod_cap_upper">
         <inertial>
@@ -174,5 +167,5 @@
         </inertial>
     </xacro:macro>
-    <!-- Lower rod-cap (×6) -->
+    <!-- Lower rod-cap — rod_cap_7 … rod_cap_12 -->
     <xacro:macro name="inertial_rod_cap_lower">
         <inertial>
@@ -189,5 +182,5 @@
         </inertial>
     </xacro:macro>
-    <!-- Lower pivot arm (×3) -->
+    <!-- Lower pivot arm — pivot_arm_4 / 5 / 6 -->
     <xacro:macro name="inertial_pivot_arm_lower">
         <inertial>
@@ -204,22 +197,20 @@
         </inertial>
     </xacro:macro>
-    <!-- STS circular horn / bevel pinion (×2) — driven (differential_pinion_joint_1/2 children) -->
+    <!-- Bevel pinion (×2) -->
     <xacro:macro name="inertial_sts_circular_horn">
         <inertial>
-            <mass>0.0039017949</mass>
-            <pose>0.0012497970 0 0 0 0 0</pose>
-            <inertia>
-                <ixx>1.4960e-07</ixx>
-                <ixy>0</ixy>
-                <ixz>0</ixz>
-                <iyy>7.8203e-08</iyy>
-                <iyz>0</iyz>
-                <izz>7.8203e-08</izz>
-            </inertia>
-        </inertial>
-    </xacro:macro>
-    <!-- ══════════════════════════════════════════════════════════
-         UTILITY MACROS
-    ══════════════════════════════════════════════════════════ -->
+            <mass>0.0039017949297462306</mass>
+            <pose>0.0012497970049005348 -1.622119909634578e-13 1.2469089650196687e-18 0.0 0.0 0.0</pose>
+            <inertia>
+                <ixx>1.4960205895115634e-07</ixx>
+                <iyy>7.820278679498025e-08</iyy>
+                <izz>7.820278739942979e-08</izz>
+                <ixy>1.683419393865418e-19</ixy>
+                <iyz>-4.583138977911326e-23</iyz>
+                <ixz>2.9791196117973993e-23</ixz>
+            </inertia>
+        </inertial>
+    </xacro:macro>
+    <!-- UTILITY MACROS -->
     <!-- mesh_geometry -->
     <xacro:macro name="mesh_geometry" params="file">
@@ -231,5 +222,5 @@
         </geometry>
     </xacro:macro>
-    <!-- fixed_joint -->
+    <!-- fixed_joint — type="fixed" with no pose element.    -->
     <xacro:macro name="fixed_joint" params="name parent child">
         <joint name="${name}" type="fixed">
@@ -238,5 +229,5 @@
         </joint>
     </xacro:macro>
-    <!-- revolute_joint -->
+    <!-- revolute_joint — type="revolute" -->
     <xacro:macro name="revolute_joint" params="name parent child ax ay az">
         <joint name="${name}" type="revolute">
@@ -248,12 +239,10 @@
         </joint>
     </xacro:macro>
-    <!-- ══════════════════════════════════════════════════════════
-         LINK MACROS
-    ══════════════════════════════════════════════════════════ -->
-    <!-- servo_mount_link (×3) -->
+    <!-- LINK MACROS -->
+    <!-- servo_mount_link -->
     <xacro:macro name="servo_mount_link" params="n px py pz roll pitch yaw">
         <link name="servo_mount_${n}">
             <self_collide>false</self_collide>
-            <pose relative_to="delta_base">${px} ${py} ${pz} ${roll} ${pitch} ${yaw}</pose>
+            <pose relative_to="delta_base-v1">${px} ${py} ${pz} ${roll} ${pitch} ${yaw}</pose>
             <xacro:inertial_servo_mount/>
             <visual name="servo_mount_${n}_visual">
@@ -263,11 +252,11 @@
         </link>
     </xacro:macro>
-    <!-- servo_link (×3) -->
+    <!-- servo_link -->
     <xacro:macro name="servo_link" params="n">
         <link name="servo_${n}">
             <self_collide>false</self_collide>
-            <pose relative_to="servo_mount_${n}">0 0 -0.0213 ${pi/2} ${pi/2} 0</pose>
+            <pose relative_to="servo_mount_${n}">0 0.0 -0.0213 ${pi/2} ${pi/2} 0</pose>
             <xacro:inertial_servo/>
-            <visual name="servo_${n}_visual">
+            <visual name="servo_${n}">
                 <xacro:mesh_geometry file="servo.stl"/>
                 <xacro:material_black_abs/>
@@ -275,5 +264,5 @@
         </link>
     </xacro:macro>
-    <!-- servo_horn_link (×3) -->
+    <!-- servo_horn_link -->
     <xacro:macro name="servo_horn_link" params="n">
         <link name="servo_${n}_horn">
@@ -288,5 +277,5 @@
         </link>
     </xacro:macro>
-    <!-- servo_free_horn_link (×3) -->
+    <!-- servo_free_horn_link -->
     <xacro:macro name="servo_free_horn_link" params="n">
         <link name="servo_${n}_free_horn">
@@ -301,11 +290,11 @@
         </link>
     </xacro:macro>
-    <!-- bicep_link (×3) -->
+    <!-- bicep_link -->
     <xacro:macro name="bicep_link" params="n">
-        <link name="bicep_${n}">
+        <link name="bicep${n}">
             <self_collide>false</self_collide>
             <pose relative_to="servo_${n}_horn">0 0 0 0 0 ${-pi/2}</pose>
             <xacro:inertial_bicep/>
-            <visual name="bicep_${n}_visual">
+            <visual name="bicep${n}_visual">
                 <xacro:mesh_geometry file="bicep.stl"/>
                 <xacro:material_white_pla/>
@@ -313,5 +302,5 @@
         </link>
     </xacro:macro>
-    <!-- pivot_arm_upper_link (×3) -->
+    <!-- pivot_arm_upper_link -->
     <xacro:macro name="pivot_arm_upper_link" params="n px py pz roll pitch yaw">
         <link name="pivot_arm_${n}">
@@ -325,5 +314,5 @@
         </link>
     </xacro:macro>
-    <!-- rod_cap_upper_link (×6) -->
+    <!-- rod_cap_upper_link -->
     <xacro:macro name="rod_cap_upper_link" params="n relative_to z_offset">
         <link name="rod_cap_${n}">
@@ -338,5 +327,5 @@
         </link>
     </xacro:macro>
-    <!-- forearm_link (×6) -->
+    <!-- forearm_link -->
     <xacro:macro name="forearm_link" params="n relative_to">
         <link name="forearm_${n}">
@@ -350,5 +339,5 @@
         </link>
     </xacro:macro>
-    <!-- rod_cap_lower_link (×6) -->
+    <!-- rod_cap_lower_link -->
     <xacro:macro name="rod_cap_lower_link" params="n relative_to roll">
         <link name="rod_cap_${n}">
@@ -362,5 +351,5 @@
         </link>
     </xacro:macro>
-    <!-- pivot_arm_lower_link (×3) -->
+    <!-- pivot_arm_lower_link -->
     <xacro:macro name="pivot_arm_lower_link" params="n relative_to">
         <link name="pivot_arm_${n}">
@@ -375,26 +364,19 @@
         </link>
     </xacro:macro>
-    <!-- detach_aux_link (×3) — massless aux links for DetachableJoint -->
-    <xacro:macro name="detach_aux_link" params="n">
-        <link name="rod_cap_${n}_aux">
-            <self_collide>false</self_collide>
-            <pose relative_to="rod_cap_${n}">0.0093 -0.005 0 0 0 0</pose>
-        </link>
-    </xacro:macro>
-    <!-- end_effector_side_plate_link (×2) -->
+    <!--end_effector_side_plate_link-->
     <xacro:macro name="end_effector_side_plate_link" params="n relative_to">
         <link name="end_effector_side_plate_${n}">
             <self_collide>false</self_collide>
-            <pose relative_to="${relative_to}">${((-1)**n) * 0.0346} 0.025 0 0 ${(n-2) * pi} 0</pose>
-            <inertial>
-                <mass>0.0225974194</mass>
-                <pose>-0.00016121771 -0.00081452055 0 0 0 0</pose>
-                <inertia>
-                    <ixx>1.0070887078e-05</ixx>
-                    <ixy>-1.8768434113e-08</ixy>
-                    <ixz>0</ixz>
-                    <iyy>3.3684942311e-06</iyy>
-                    <iyz>0</iyz>
-                    <izz>7.0797253681e-06</izz>
+            <pose relative_to="${relative_to}">${((-1)**n) * 0.0346} 0.025 0  0 ${(n-2) * pi} 0</pose>
+            <inertial>
+                <mass>0.022597419423661277</mass>
+                <pose>-0.00016121770501891622 -0.0008145205514591019 1.2212521563574412e-14 0.0 0.0 0.0</pose>
+                <inertia>
+                    <ixx>1.0070887077865201e-05</ixx>
+                    <iyy>3.3684942310930237e-06</iyy>
+                    <izz>7.079725368086249e-06</izz>
+                    <ixy>-1.8768434113228535e-08</ixy>
+                    <iyz>6.0129338666995994e-18</iyz>
+                    <ixz>-2.5052368945177017e-19</ixz>
                 </inertia>
             </inertial>
@@ -404,19 +386,18 @@
         </link>
     </xacro:macro>
-    <!-- differential_servo_link (×2) — driven (differential_pinion_joint_1/2 parents) -->
     <xacro:macro name="differential_servo" params="n relative_to">
         <link name="differential_servo_${n}">
             <self_collide>false</self_collide>
-            <pose relative_to="${relative_to}">0.0024 0.005 0 ${pi/2} ${pi/2} 0</pose>
-            <inertial>
-                <mass>0.0620599988</mass>
-                <pose>0 0.0079594816 0.0055633688 0 0 0</pose>
-                <inertia>
-                    <ixx>6.9884428428e-06</ixx>
-                    <ixy>0</ixy>
-                    <ixz>0</ixz>
-                    <iyy>3.6553944820e-06</iyy>
-                    <iyz>-3.4792797513e-08</iyz>
-                    <izz>4.7934769497e-06</izz>
+            <pose relative_to="${relative_to}">0.0024  0.005 0 ${pi/2} ${pi/2} 0</pose>
+            <inertial>
+                <mass>0.06205999879006312</mass>
+                <pose>5.440072487533238e-15 0.00795948162757361 0.005563368804401614 0.0 0.0 0.0</pose>
+                <inertia>
+                    <ixx>6.988442842844299e-06</ixx>
+                    <iyy>3.6553944820485586e-06</iyy>
+                    <izz>4.7934769497030256e-06</izz>
+                    <ixy>5.20881887690237e-18</ixy>
+                    <iyz>-3.479279751288407e-08</iyz>
+                    <ixz>2.054868248794087e-18</ixz>
                 </inertia>
             </inertial>
@@ -427,17 +408,4 @@
         </link>
     </xacro:macro>
-    <!-- sts_circular_horn_link (×2) — driven (differential_pinion_joint_1/2 children) -->
-    <xacro:macro name="sts_circular_horn_link" params="n relative_to">
-        <link name="sts_circular_horn_${n}">
-            <self_collide>false</self_collide>
-            <pose relative_to="${relative_to}">0 -0.0110 0 0 0 ${pi/2}</pose>
-            <xacro:inertial_sts_circular_horn/>
-            <visual name="sts_circular_horn_${n}_visual">
-                <xacro:mesh_geometry file="sts_circular_horn.stl"/>
-                <xacro:material_black_pla/>
-            </visual>
-        </link>
-    </xacro:macro>
-    <!-- end_effector_pinion_link (×2) — driven -->
     <xacro:macro name="end_effector_pinion" params="n relative_to">
         <link name="end_effector_pinion_${n}">
@@ -445,13 +413,13 @@
             <pose relative_to="${relative_to}">0.002 0 0 0 0 ${pi/2}</pose>
             <inertial>
-                <mass>0.0031576875</mass>
-                <pose>0 0.0080716975 0 0 0 0</pose>
-                <inertia>
-                    <ixx>1.2058613504e-07</ixx>
-                    <ixy>0</ixy>
-                    <ixz>0</ixz>
-                    <iyy>1.2922906781e-07</iyy>
-                    <iyz>0</iyz>
-                    <izz>1.2058567290e-07</izz>
+                <mass>0.003157687504521257</mass>
+                <pose>-5.365483655606078e-09 0.008071697510068476 -1.9417273873692396e-09 0.0 0.0 0.0</pose>
+                <inertia>
+                    <ixx>1.2058613504333728e-07</ixx>
+                    <iyy>1.2922906780614413e-07</iyy>
+                    <izz>1.2058567289965568e-07</izz>
+                    <ixy>-6.497217694519726e-14</ixy>
+                    <iyz>1.0051734377178594e-13</iyz>
+                    <ixz>3.427645062296904e-14</ixz>
                 </inertia>
             </inertial>
@@ -462,5 +430,5 @@
         </link>
     </xacro:macro>
-    <!-- virtual_pivot_link (×3) -->
+    <!-- virtual_pivot_link -->
     <xacro:macro name="virtual_pivot_link" params="n relative_to">
         <link name="virtual_pivot_${n}">
@@ -469,8 +437,5 @@
         </link>
     </xacro:macro>
-    <!-- ══════════════════════════════════════════════════════════
-         JOINT MACROS
-    ══════════════════════════════════════════════════════════ -->
-    <!-- motor_joint_set — driven revolute + mimic free-horn (×3) -->
+    <!-- motor_joint_set -->
     <xacro:macro name="motor_joint_set" params="n">
         <joint name="motor_joint_${n}" type="revolute">
@@ -493,7 +458,5 @@
         </joint>
     </xacro:macro>
-    <!-- ══════════════════════════════════════════════════════════
-         MODEL
-    ══════════════════════════════════════════════════════════ -->
+    <!-- MODEL -->
     <model name="delta_robot">
         <!-- World anchor -->
@@ -529,8 +492,8 @@
                 </inertia>
             </inertial>
-            <collision name="frame_collision">
+            <collision name="Frame_collision">
                 <xacro:mesh_geometry file="frame.stl"/>
             </collision>
-            <visual name="frame_visual">
+            <visual name="Frame_visual">
                 <xacro:mesh_geometry file="frame.stl"/>
                 <xacro:material_black_aluminium/>
@@ -538,5 +501,5 @@
         </link>
         <!-- Delta base plate -->
-        <link name="delta_base">
+        <link name="delta_base-v1">
             <self_collide>false</self_collide>
             <pose>0 0 -0.01 0 0 0</pose>
@@ -553,44 +516,44 @@
                 </inertia>
             </inertial>
-            <visual name="delta_base_visual">
+            <visual name="delta_base-v1_visual">
                 <xacro:mesh_geometry file="delta_base-v1.stl"/>
                 <xacro:material_aluminium/>
             </visual>
         </link>
-        <!-- ─── Arm 1 ─── -->
+        <!-- Arm 1 -->
         <xacro:servo_mount_link n="1"
-            px=" 0.0787"  py=" 0.0"      pz="0.01"
-            roll="${-pi/2}" pitch="0"    yaw="${pi/2}"/>
+            px=" 0.0787"  py="0"       pz="0.01"
+            roll="${-pi/2}" pitch="0"  yaw="${pi/2}"/>
         <xacro:servo_link           n="1"/>
         <xacro:servo_horn_link      n="1"/>
         <xacro:servo_free_horn_link n="1"/>
         <xacro:bicep_link           n="1"/>
-        <!-- ─── Arm 2 ─── -->
+        <!-- Arm 2 -->
         <xacro:servo_mount_link n="2"
-            px="-0.03935" py=" 0.06816"  pz="0.01"
-            roll="${-pi/2}" pitch="0"    yaw="${-5*pi/6}"/>
+            px="-0.03935"  py=" 0.06816"  pz="0.01"
+            roll="${-pi/2}" pitch="0"     yaw="${-5*pi/6}"/>
         <xacro:servo_link           n="2"/>
         <xacro:servo_horn_link      n="2"/>
         <xacro:servo_free_horn_link n="2"/>
         <xacro:bicep_link           n="2"/>
-        <!-- ─── Arm 3 ─── -->
+        <!-- Arm 3 -->
         <xacro:servo_mount_link n="3"
-            px="-0.03935" py="-0.06816"  pz="0.01"
-            roll="${-pi/2}" pitch="0"    yaw="${-pi/6}"/>
+            px="-0.03935"  py="-0.06816"  pz="0.01"
+            roll="${-pi/2}" pitch="0"     yaw="${-pi/6}"/>
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