Commit message: Add TF error plotting and visualization tools
- Implemented `tf_error_plotter.py` for real-time plotting of TF errors between commanded and actual end-effector positions.
- Created a new ROS package `delta_telemetry` with necessary configuration files (`package.xml`, `setup.py`, `setup.cfg`).
- Added resource directory for package resources.
- Included test files for copyright, flake8, and PEP257 compliance.
- Introduced `plot_ee_tf.py` for real-time TF visualization using PyQtGraph, supporting multiple views (2D and 3D) and RPY time-series.
- Enhanced GUI controls for freezing and saving plots.

File: delta_robot_description/models/model_high.sdf.xacro (robot description, xacro)
@@ -12,5 +12,5 @@
             <ambient>0.2  0.2  0.2  1</ambient>
             <diffuse>0.3  0.3  0.3  1</diffuse>
-            <specular>0.95 0.95 0.95 1</specular>
+            <specular>1.0  1.0  1.0  1</specular>
         </material>
     </xacro:macro>
@@ -36,11 +36,4 @@
         </material>
     </xacro:macro>
-    <xacro:macro name="material_grey_pla">
-        <material>
-            <ambient>0.15 0.15 0.15 1</ambient>
-            <diffuse>0.4  0.4  0.4  1</diffuse>
-            <specular>0.05 0.05 0.05 1</specular>
-        </material>
-    </xacro:macro>
     <xacro:macro name="material_black_pla">
         <material>
@@ -48,4 +41,11 @@
             <diffuse>0.1  0.1  0.1  1</diffuse>
             <specular>0.05 0.05 0.05 1</specular>
+        </material>
+    </xacro:macro>
+    <xacro:macro name="material_orange_pla">
+        <material>
+            <ambient>0.4  0.15 0.0  1</ambient>
+            <diffuse>1.0  0.4  0.0  1</diffuse>
+            <specular>0.1  0.1  0.1  1</specular>
         </material>
     </xacro:macro>
@@ -321,5 +321,5 @@
             <visual name="pivot_arm_${n}_visual">
                 <xacro:mesh_geometry file="pivot_arm.stl"/>
-                <xacro:material_grey_pla/>
+                <xacro:material_white_pla/>
             </visual>
         </link>
@@ -371,5 +371,5 @@
                 <pose>0 0 -0.016 0 0 0</pose>
                 <xacro:mesh_geometry file="pivot_arm.stl"/>
-                <xacro:material_grey_pla/>
+                <xacro:material_white_pla/>
             </visual>
         </link>
@@ -401,4 +401,5 @@
             <visual name="end_effector_side_plate_${n}_visual">
                 <xacro:mesh_geometry file="end_effector_side_plate.stl"/>
+                <xacro:material_orange_pla/>
             </visual>
         </link>
@@ -480,4 +481,5 @@
                 <xyz>0 1 0</xyz>
             </axis>
+            <limit effort="2.0" velocity="11.1" lower="-3.14159" upper="3.14159"/>
         </joint>
         <joint name="motor_joint_${n}_free" type="revolute">
@@ -499,4 +501,5 @@
         <!-- World anchor -->
         <link name="world_link">
+            <pose>0 0 0 0 0 ${pi/2}</pose>
             <self_collide>false</self_collide>
             <inertial>
@@ -516,5 +519,5 @@
             <self_collide>false</self_collide>
             <static>true</static>
-            <pose>0 0 -0.059454 0 0 0</pose>
+            <pose relative_to="world_link">0 0 -0.059454 0 0 0</pose>
             <inertial>
                 <pose>0 0 0 0 0 0</pose>
@@ -640,5 +643,5 @@
             <visual name="end_effector_visual">
                 <xacro:mesh_geometry file="end_effector.stl"/>
-                <xacro:material_black_pla/>
+                <xacro:material_orange_pla/>
             </visual>
         </link>
@@ -663,5 +666,5 @@
             <visual name="end_effector_base_plate_visual">
                 <xacro:mesh_geometry file="end_effector_base_plate.stl"/>
-                <xacro:material_grey_pla/>
+                <xacro:material_orange_pla/>
             </visual>
         </link>
@@ -697,5 +700,5 @@
             <visual name="middle_shaft_visual">
                 <xacro:mesh_geometry file="middle_shaft.stl"/>
-                <xacro:material_grey_pla/>
+                <xacro:material_black_pla/>
             </visual>
         </link>
@@ -721,4 +724,27 @@
                 <xacro:material_black_pla/>
             </visual>
+        </link>
+        <link name="cube">
+            <pose relative_to="bevel_gear_ee"> 0 -0.03775 0  ${-pi/2} 0 0</pose>
+            <inertial>
+                <mass>0.2190086521864867</mass>
+                <pose>-0.0007571147448307052 -0.0004725953633605644 0.00028984668097712914 0.0 0.0 0.0</pose>
+                <inertia>
+                    <ixx>6.725551979614924e-05</ixx>
+                    <iyy>6.782851202234727e-05</iyy>
+                    <izz>6.74186794018338e-05</izz>
+                    <ixy>8.080306097808026e-08</ixy>
+                    <iyz>2.2480222406133124e-07</iyz>
+                    <ixz>-1.1044106726896244e-07</ixz>
+                </inertia>
+            </inertial>
+            <visual name="cube_visual">
+                <xacro:mesh_geometry file="cube.stl"/>
+                <xacro:material_black_pla/>
+            </visual>
+        </link>
+        <link name="end_effector_pin">
+            <self_collide>false</self_collide>
+            <pose relative_to="cube">0 0 0 ${pi/2} ${pi/2} ${pi} </pose>
         </link>
         <!-- ─── Virtual pivot constraints ─── -->
@@ -820,9 +846,11 @@
         <xacro:fixed_joint    name="side_plate_2_to_diff_servo_2" parent="end_effector_side_plate_2" child="differential_servo_2"/>
         <xacro:fixed_joint    name="virtual_middle_shaft_to_middle_shaft"     parent="virtual_middle_shaft"     child="middle_shaft"/>
-        <xacro:revolute_joint name="differential_EE_joint"        parent="middle_shaft"            child="bevel_gear_ee"          ax="0" ay="1" az="0"/>
+        <xacro:revolute_joint name="differential_EE_joint"        parent="middle_shaft"            child="bevel_gear_ee"          ax="0" ay="-1" az="0"/>
         <xacro:revolute_joint name="differential_pinion_joint_1"  parent="differential_servo_1"    child="sts_circular_horn_1"    ax="1" ay="0"  az="0"/>
         <xacro:revolute_joint name="differential_pinion_joint_2"  parent="differential_servo_2"    child="sts_circular_horn_2"    ax="1" ay="0"  az="0"/>
         <xacro:fixed_joint    name="sts_horn_1_to_ee_pinion_1"    parent="sts_circular_horn_1"     child="end_effector_pinion_1"/>
         <xacro:fixed_joint    name="sts_horn_2_to_ee_pinion_2"    parent="sts_circular_horn_2"     child="end_effector_pinion_2"/>
+        <xacro:fixed_joint    name="bevel_gear_ee_to_cube" parent="bevel_gear_ee" child="cube"/>
+        <xacro:fixed_joint    name="cube_to_end_effector_pin" parent="cube" child="end_effector_pin"/>
         <!-- ══════════════════════════════════════════════════════════
              ROS 2 CONTROL

Commit message: Test2

File: delta_robot_description/models/model_high.sdf.xacro (robot description, xacro)
@@ -857,45 +857,59 @@
         ══════════════════════════════════════════════════════════ -->
         <ros2_control name="GazeboSimSystem" type="system">
-            <hardware>
-                <plugin>gz_ros2_control/GazeboSimSystem</plugin>
-            </hardware>
-            <!-- Motor joints -->
-            <joint name="motor_joint_1">
-                <command_interface name="position"/>
-                <state_interface   name="position"/>
-                <state_interface   name="velocity"/>
-            </joint>
-            <joint name="motor_joint_2">
-                <command_interface name="position"/>
-                <state_interface   name="position"/>
-                <state_interface   name="velocity"/>
-            </joint>
-            <joint name="motor_joint_3">
-                <command_interface name="position"/>
-                <state_interface   name="position"/>
-                <state_interface   name="velocity"/>
-            </joint>
-            <!-- Differential joints -->
-            <joint name="differential_pinion_joint_1">
-                <command_interface name="position"/>
-                <state_interface   name="position"/>
-                <state_interface   name="velocity"/>
-            </joint>
-            <joint name="differential_pinion_joint_2">
-                <command_interface name="position"/>
-                <state_interface   name="position"/>
-                <state_interface   name="velocity"/>
-            </joint>
-            <joint name="differential_T_joint">
-                <command_interface name="position"/>
-                <state_interface   name="position"/>
-                <state_interface   name="velocity"/>
-            </joint>
-            <joint name="differential_EE_joint">
-                <command_interface name="position"/>
-                <state_interface   name="position"/>
-                <state_interface   name="velocity"/>
-            </joint>
-        </ros2_control>
+    <hardware>
+        <plugin>gz_ros2_control/GazeboSimSystem</plugin>
+    </hardware>
+    <!-- Motor joints -->
+    <joint name="motor_joint_1">
+        <command_interface name="position"/>
+        <state_interface name="position">
+            <param name="initial_value">0.0</param>
+        </state_interface>
+        <state_interface name="velocity"/>
+    </joint>
+    <joint name="motor_joint_2">
+        <command_interface name="position"/>
+        <state_interface name="position">
+            <param name="initial_value">0.0</param>
+        </state_interface>
+        <state_interface name="velocity"/>
+    </joint>
+    <joint name="motor_joint_3">
+        <command_interface name="position"/>
+        <state_interface name="position">
+            <param name="initial_value">0.0</param>
+        </state_interface>
+        <state_interface name="velocity"/>
+    </joint>
+    <!-- Differential joints -->
+    <joint name="differential_pinion_joint_1">
+        <command_interface name="position"/>
+        <state_interface name="position">
+            <param name="initial_value">0.0</param>
+        </state_interface>
+        <state_interface name="velocity"/>
+    </joint>
+    <joint name="differential_pinion_joint_2">
+        <command_interface name="position"/>
+        <state_interface name="position">
+            <param name="initial_value">0.0</param>
+        </state_interface>
+        <state_interface name="velocity"/>
+    </joint>
+    <joint name="differential_T_joint">
+        <command_interface name="position"/>
+        <state_interface name="position">
+            <param name="initial_value">0.0</param>
+        </state_interface>
+        <state_interface name="velocity"/>
+    </joint>
+    <joint name="differential_EE_joint">
+        <command_interface name="position"/>
+        <state_interface name="position">
+            <param name="initial_value">0.0</param>
+        </state_interface>
+        <state_interface name="velocity"/>
+    </joint>
+</ros2_control>
         <!-- ══════════════════════════════════════════════════════════
              PLUGINS
